File: PCB/reflowControllerV2.kicad_pcb (KiCad board)
At the start: 4 copper layers, 43 x 89 mm, 99 parts, among them J10 NEXTION_OB, J11 PWR, J12 A-1JB, J2 SSR2, J3 SSR1, J4 FAN1, J5 FAN2, J6 T1, J7 T2, J8 SWD, J9 NEXTION_FRONT, Q1 BSS316NH6327, Q2 BSS316NH6327, Q3 BSS316NH6327, Q4 BSS316NH6327, Q5 BSS316NH6327, SW1 B3F-4055, U1 918-468K2029E50001, U10 ZD24C128A, U2 918-468K2029E50001, U3 AMS1117-3.3, U4 STM32WBxx_QFN48, U5 USBLC6-2SC6, U6 USBLC6-2SC6, U7 CH340G, U8 MAX31855KASA, U9 MAX31855KASA, Y1 NX2016_32MHz, Y2 NX2012_32K768Hz, Y3 12M

Commit message: Few changes
Connections:
- net Net-(U1-PadA4) renamed /USB_VBUS
- net Net-(U2-PadA4) renamed /USB_VBUS2
Changed lines of the file:
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@@
 (kicad_pcb (version 20211014) (generator pcbnew)
   (general
-    (thickness 4.69)
+    (thickness 1.66)
   )
   (paper "A4")
@@
       (layer "F.Mask" (type "Top Solder Mask") (thickness 0.01))
       (layer "F.Cu" (type "copper") (thickness 0.035))
-      (layer "dielectric 1" (type "core") (thickness 1.51) (material "FR4") (epsilon_r 4.5) (loss_tangent 0.02))
+      (layer "dielectric 1" (type "core") (thickness 0.7) (material "FR4") (epsilon_r 4.5) (loss_tangent 0.02))
       (layer "In1.Cu" (type "copper") (thickness 0.035))
-      (layer "dielectric 2" (type "prepreg") (thickness 1.51) (material "FR4") (epsilon_r 4.5) (loss_tangent 0.02))
+      (layer "dielectric 2" (type "prepreg") (thickness 0.1) (material "FR4") (epsilon_r 4.5) (loss_tangent 0.02))
       (layer "In2.Cu" (type "copper") (thickness 0.035))
-      (layer "dielectric 3" (type "core") (thickness 1.51) (material "FR4") (epsilon_r 4.5) (loss_tangent 0.02))
+      (layer "dielectric 3" (type "core") (thickness 0.7) (material "FR4") (epsilon_r 4.5) (loss_tangent 0.02))
       (layer "B.Cu" (type "copper") (thickness 0.035))
       (layer "B.Mask" (type "Bottom Solder Mask") (thickness 0.01))
@@
   (net 44 "/USB1_D+")
   (net 45 "/ST_USB_D+")
-  (net 46 "Net-(U1-PadA4)")
+  (net 46 "/USB_VBUS")
   (net 47 "/ST_USB_D-")
   (net 48 "/UART_USB_D+")
-  (net 49 "Net-(U2-PadA4)")
+  (net 49 "/USB_VBUS2")
   (net 50 "/UART_USB_D-")
   (net 51 "/LPUART1_RX")
@@
       (net 45 "/ST_USB_D+") (pinfunction "I/O2") (pintype "passive"))
     (pad "5" smd roundrect (at 1.1375 0 180) (size 1.325 0.6) (layers "F.Cu" "F.Paste" "F.Mask") (roundrect_rratio 0.25)
-      (net 46 "Net-(U1-PadA4)") (pinfunction "VBUS") (pintype "passive"))
+      (net 46 "/USB_VBUS") (pinfunction "VBUS") (pintype "passive"))
     (pad "6" smd roundrect (at 1.1375 -0.95 180) (size 1.325 0.6) (layers "F.Cu" "F.Paste" "F.Mask") (roundrect_rratio 0.25)
       (net 47 "/ST_USB_D-") (pinfunction "I/O1") (pintype "passive"))
@@
       (net 48 "/UART_USB_D+") (pinfunction "I/O2") (pintype "passive"))
     (pad "5" smd roundrect (at 1.1375 0 180) (size 1.325 0.6) (layers "F.Cu" "F.Paste" "F.Mask") (roundrect_rratio 0.25)
-      (net 49 "Net-(U2-PadA4)") (pinfunction "VBUS") (pintype "passive"))
+      (net 49 "/USB_VBUS2") (pinfunction "VBUS") (pintype "passive"))
     (pad "6" smd roundrect (at 1.1375 -0.95 180) (size 1.325 0.6) (layers "F.Cu" "F.Paste" "F.Mask") (roundrect_rratio 0.25)
       (net 50 "/UART_USB_D-") (pinfunction "I/O1") (pintype "passive"))
@@
       (net 4 "GND") (pinfunction "GND") (pintype "power_in"))
     (pad "A4" thru_hole circle (at 0.58 1.84 90) (size 0.7 0.7) (drill 0.4) (layers *.Cu *.Mask)
-      (net 49 "Net-(U2-PadA4)") (pinfunction "VBUS") (pintype "power_in"))
+      (net 49 "/USB_VBUS2") (pinfunction "VBUS") (pintype "power_in"))
     (pad "A5" thru_hole circle (at 0.58 0.84 90) (size 0.7 0.7) (drill 0.4) (layers *.Cu *.Mask)
       (net 66 "unconnected-(U2-PadA5)") (pinfunction "CC1") (pintype "bidirectional+no_connect"))
@@
       (net 68 "/USB2_D-") (pinfunction "DN1") (pintype "bidirectional"))
     (pad "A9" thru_hole circle (at 0.58 -2.16 90) (size 0.7 0.7) (drill 0.4) (layers *.Cu *.Mask)
-      (net 49 "Net-(U2-PadA4)") (pinfunction "VBUS") (pintype "power_in"))
+      (net 49 "/USB_VBUS2") (pinfunction "VBUS") (pintype "power_in"))
     (pad "A12" thru_hole circle (at 0.58 -3.16 90) (size 0.7 0.7) (drill 0.4) (layers *.Cu *.Mask)
       (net 4 "GND") (pinfunction "GND") (pintype "power_in"))
@@
       (net 4 "GND") (pinfunction "GND") (pintype "power_in"))
     (pad "B4" thru_hole circle (at -0.58 -1.84 90) (size 0.7 0.7) (drill 0.4) (layers *.Cu *.Mask)
-      (net 49 "Net-(U2-PadA4)") (pinfunction "VBUS") (pintype "power_in"))
+      (net 49 "/USB_VBUS2") (pinfunction "VBUS") (pintype "power_in"))
     (pad "B5" thru_hole circle (at -0.58 -0.84 90) (size 0.7 0.7) (drill 0.4) (layers *.Cu *.Mask)
       (net 69 "unconnected-(U2-PadB5)") (pinfunction "CC2") (pintype "bidirectional+no_connect"))
@@
       (net 68 "/USB2_D-") (pinfunction "DN2") (pintype "bidirectional"))
     (pad "B9" thru_hole circle (at -0.58 2.16 90) (size 0.7 0.7) (drill 0.4) (layers *.Cu *.Mask)
-      (net 49 "Net-(U2-PadA4)") (pinfunction "VBUS") (pintype "power_in"))
+      (net 49 "/USB_VBUS2") (pinfunction "VBUS") (pintype "power_in"))
     (pad "B12" thru_hole circle (at -0.58 3.16 90) (size 0.7 0.7) (drill 0.4) (layers *.Cu *.Mask)
       (net 4 "GND") (pinfunction "GND") (pintype "power_in"))
@@
       (net 4 "GND") (pinfunction "GND") (pintype "power_in"))
     (pad "A4" thru_hole circle (at 0.58 1.84 90) (size 0.7 0.7) (drill 0.4) (layers *.Cu *.Mask)
-      (net 46 "Net-(U1-PadA4)") (pinfunction "VBUS") (pintype "power_in"))
+      (net 46 "/USB_VBUS") (pinfunction "VBUS") (pintype "power_in"))
     (pad "A5" thru_hole circle (at 0.58 0.84 90) (size 0.7 0.7) (drill 0.4) (layers *.Cu *.Mask)
       (net 64 "unconnected-(U1-PadA5)") (pinfunction "CC1") (pintype "bidirectional+no_connect"))
@@
       (net 43 "/USB1_D-") (pinfunction "DN1") (pintype "bidirectional"))
     (pad "A9" thru_hole circle (at 0.58 -2.16 90) (size 0.7 0.7) (drill 0.4) (layers *.Cu *.Mask)
-      (net 46 "Net-(U1-PadA4)") (pinfunction "VBUS") (pintype "power_in"))
+      (net 46 "/USB_VBUS") (pinfunction "VBUS") (pintype "power_in"))
     (pad "A12" thru_hole circle (at 0.58 -3.16 90) (size 0.7 0.7) (drill 0.4) (layers *.Cu *.Mask)
       (net 4 "GND") (pinfunction "GND") (pintype "power_in"))
@@
       (net 4 "GND") (pinfunction "GND") (pintype "power_in"))
     (pad "B4" thru_hole circle (at -0.58 -1.84 90) (size 0.7 0.7) (drill 0.4) (layers *.Cu *.Mask)
-      (net 46 "Net-(U1-PadA4)") (pinfunction "VBUS") (pintype "power_in"))
+      (net 46 "/USB_VBUS") (pinfunction "VBUS") (pintype "power_in"))
     (pad "B5" thru_hole circle (at -0.58 -0.84 90) (size 0.7 0.7) (drill 0.4) (layers *.Cu *.Mask)
       (net 65 "unconnected-(U1-PadB5)") (pinfunction "CC2") (pintype "bidirectional+no_connect"))
@@
       (net 43 "/USB1_D-") (pinfunction "DN2") (pintype "bidirectional"))
     (pad "B9" thru_hole circle (at -0.58 2.16 90) (size 0.7 0.7) (drill 0.4) (layers *.Cu *.Mask)
-      (net 46 "Net-(U1-PadA4)") (pinfunction "VBUS") (pintype "power_in"))
+      (net 46 "/USB_VBUS") (pinfunction "VBUS") (pintype "power_in"))
     (pad "B12" thru_hole circle (at -0.58 3.16 90) (size 0.7 0.7) (drill 0.4) (layers *.Cu *.Mask)
       (net 4 "GND") (pinfunction "GND") (pintype "power_in"))
