File: PCB/reflowControllerV2.kicad_pcb (KiCad board)
At the start: 4 copper layers, 43 x 89 mm, 99 parts, among them J10 NEXTION_OB, J11 PWR, J12 A-1JB, J2 SSR2, J3 SSR1, J4 FAN1, J5 FAN2, J6 T1, J7 T2, J8 SWD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

Commit message: Few changes
Connections:
- net Net-(BZ1-Pad2) renamed /B_m
- net Net-(C30-Pad2) renamed /VFB
- net Net-(C31-Pad2) renamed /VDDA
- net Net-(D1-Pad1) renamed /ON_LED
- net Net-(JP1-Pad1) renamed /BOOT0
- net Net-(L3-Pad2) renamed /VLX
Routing:
- net GND: vias 191 -> 204

Commit message: Reorganized schematic
Parts:
- L4: value NF -> 0R
Connections:
- net Net-(ANT1-Pad1) renamed /RF_ANTENNA
- net Net-(C24-Pad1) renamed /RF_FILTER
- net Net-(C24-Pad2) renamed /RF_F2_IN
- net Net-(C34-Pad2) renamed /RF_F1_IN
- net Net-(C36-Pad2) renamed /RF_SMA
- net Net-(F1-Pad3) renamed /RF_OUT
