File: PCB/reflowControllerV2.kicad_sch (KiCad schematic)
At the start: 96 parts, among them J10 NEXTION_OB, J11 PWR, J12 A-1JB, J2 SSR2, J3 SSR1, J4 FAN1, J5 FAN2, J6 T1, J7 T2, J8 SWD, J9 NEXTION_FRONT, Q1 BSS316NH6327, Q2 BSS316NH6327, Q3 BSS316NH6327, Q4 BSS316NH6327, Q5 BSS316NH6327, SW1 B3F-4055, U1 918-468K2029E50001, U10 ZD24C128A, U2 918-468K2029E50001, U3 AMS1117-3.3, U4 STM32WBxx_QFN48, U5 USBLC6-2SC6, U6 USBLC6-2SC6, U7 CH340G, U8 MAX31855KASA, U9 MAX31855KASA, Y1 NX2016_32MHz, Y2 NX2012_32K768Hz, Y3 12M

Commit message: PCB finalized, Gerbers created, Firmware dir renamed
Connections:
- net USART1_RX: now also J10.2 (Pin_2), J9.2 (Pin_2); no longer J10.3 (Pin_3), J9.3 (Pin_3)
- net USART1_TX: now also J10.3 (Pin_3), J9.3 (Pin_3); no longer J10.2 (Pin_2), J9.2 (Pin_2)
Other:
- moved on the sheet: D2
Changed lines of the file:
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@@
   (no_connect (at 27.94 59.055))
   (no_connect (at 104.775 114.3))
-  (no_connect (at 149.86 -15.875))
+  (no_connect (at 154.94 46.355))
   (no_connect (at 125.095 132.08))
   (no_connect (at 125.095 129.54))
@@
     (stroke (width 0) (type default) (color 0 0 0 0))
   )
-  (wire (pts (xy 127.635 -15.875) (xy 134.62 -15.875))
+  (wire (pts (xy 132.715 46.355) (xy 139.7 46.355))
     (stroke (width 0) (type default) (color 0 0 0 0))
   )
@@
     (stroke (width 0) (type default) (color 0 0 0 0))
   )
-  (wire (pts (xy 142.24 -8.255) (xy 142.24 -6.985))
+  (wire (pts (xy 147.32 53.975) (xy 147.32 55.245))
     (stroke (width 0) (type default) (color 0 0 0 0))
   )
@@
     (stroke (width 0) (type default) (color 0 0 0 0))
   )
-  (wire (pts (xy 142.24 -24.13) (xy 142.24 -23.495))
+  (wire (pts (xy 147.32 38.1) (xy 147.32 38.735))
     (stroke (width 0) (type default) (color 0 0 0 0))
   )
@@
     (effects (font (size 1 1)) (justify left bottom))
   )
-  (label "WS_DATA" (at 127.635 -15.875 0)
+  (label "WS_DATA" (at 132.715 46.355 0)
     (effects (font (size 1 1)) (justify left bottom))
   )
@@
     (effects (font (size 1 1)) (justify left bottom))
   )
-  (label "USART1_RX" (at 200.66 53.34 0)
+  (label "USART1_RX" (at 200.66 50.8 0)
     (effects (font (size 1 1)) (justify left bottom))
   )
@@
     (effects (font (size 1 1)) (justify right bottom))
   )
-  (label "USART1_TX" (at 200.66 50.8 0)
+  (label "USART1_TX" (at 200.66 53.34 0)
     (effects (font (size 1 1)) (justify left bottom))
   )
-  (label "USART1_RX" (at 199.39 31.75 0)
+  (label "USART1_RX" (at 199.39 29.21 0)
     (effects (font (size 1 1)) (justify left bottom))
   )
@@
     (effects (font (size 1 1)) (justify left bottom))
   )
-  (label "USART1_TX" (at 199.39 29.21 0)
+  (label "USART1_TX" (at 199.39 31.75 0)
     (effects (font (size 1 1)) (justify left bottom))
   )
@@
     (pin "1")
   )
-  (symbol (lib_id "LED:WS2812B") (at 142.24 -15.875 0) (unit 1)
+  (symbol (lib_id "LED:WS2812B") (at 147.32 46.355 0) (unit 1)
     (in_bom yes) (on_board yes)
-    (property "Reference" "D2" (id 0) (at 138.43 -22.225 0))
-    (property "Value" "ST_LED" (id 1) (at 146.685 -22.225 0))
-    (property "Footprint" "LED_SMD:LED_WS2812B_PLCC4_5.0x5.0mm_P3.2mm" (id 2) (at 143.51 -8.255 0)
+    (property "Reference" "D2" (id 0) (at 143.51 40.005 0))
+    (property "Value" "ST_LED" (id 1) (at 151.765 40.005 0))
+    (property "Footprint" "LED_SMD:LED_WS2812B_PLCC4_5.0x5.0mm_P3.2mm" (id 2) (at 148.59 53.975 0)
       (effects (font (size 1.27 1.27)) (justify left top) hide)
     )
-    (property "Datasheet" "https://cdn-shop.adafruit.com/datasheets/WS2812B.pdf" (id 3) (at 144.78 -6.35 0)
+    (property "Datasheet" "https://cdn-shop.adafruit.com/datasheets/WS2812B.pdf" (id 3) (at 149.86 55.88 0)
       (effects (font (size 1.27 1.27)) (justify left top) hide)
     )
@@
     (pin "4")
   )
-  (symbol (lib_id "power:GND") (at 142.24 -6.985 0) (unit 1)
+  (symbol (lib_id "power:GND") (at 147.32 55.245 0) (unit 1)
     (in_bom yes) (on_board yes)
-    (property "Reference" "#PWR030" (id 0) (at 142.24 -0.635 0)
+    (property "Reference" "#PWR030" (id 0) (at 147.32 61.595 0)
       (effects (font (size 1.27 1.27)) hide)
     )
-    (property "Value" "GND" (id 1) (at 142.24 -3.175 0))
-    (property "Footprint" "" (id 2) (at 142.24 -6.985 0)
+    (property "Value" "GND" (id 1) (at 147.32 59.055 0))
+    (property "Footprint" "" (id 2) (at 147.32 55.245 0)
       (effects (font (size 1.27 1.27)) hide)
     )
-    (property "Datasheet" "" (id 3) (at 142.24 -6.985 0)
+    (property "Datasheet" "" (id 3) (at 147.32 55.245 0)
       (effects (font (size 1.27 1.27)) hide)
     )
@@
     (pin "4")
   )
-  (symbol (lib_id "power:+5V") (at 142.24 -24.13 0) (unit 1)
+  (symbol (lib_id "power:+5V") (at 147.32 38.1 0) (unit 1)
     (in_bom yes) (on_board yes)
-    (property "Reference" "#PWR069" (id 0) (at 142.24 -20.32 0)
+    (property "Reference" "#PWR069" (id 0) (at 147.32 41.91 0)
       (effects (font (size 1.27 1.27)) hide)
     )
-    (property "Value" "+5V" (id 1) (at 142.24 -27.94 0))
-    (property "Footprint" "" (id 2) (at 142.24 -24.13 0)
+    (property "Value" "+5V" (id 1) (at 147.32 34.29 0))
+    (property "Footprint" "" (id 2) (at 147.32 38.1 0)
       (effects (font (size 1.27 1.27)) hide)
     )
-    (property "Datasheet" "" (id 3) (at 142.24 -24.13 0)
+    (property "Datasheet" "" (id 3) (at 147.32 38.1 0)
       (effects (font (size 1.27 1.27)) hide)
     )

Commit message: Few changes
Connections:
- net USB_VBUS2: now reaches U2.A4 (VBUS), U2.A9 (VBUS), U2.B4 (VBUS), U2.B9 (VBUS), U6.5 (VBUS)
- net USB_VBUS: now reaches U1.A4 (VBUS), U1.A9 (VBUS), U1.B4 (VBUS), U1.B9 (VBUS), U5.5 (VBUS)
Other:
- company: (none) -> lukas-walczak@web.de
Changed lines of the file:
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@@
     (date "2022-04-21")
     (rev "2.0")
+    (company "lukas-walczak@web.de")
+    (comment 1 "STm32WB based toaster oven controller")
   )
   (junction (at 40.005 23.495) (diameter 0) (color 0 0 0 0)
@@
     (effects (font (size 1 1)) (justify right bottom))
   )
+  (label "USB_VBUS" (at 48.26 18.415 0)
+    (effects (font (size 1.27 1.27)) (justify left bottom))
+  )
   (label "T2_CS" (at 92.71 31.75 0)
     (effects (font (size 1 1)) (justify left bottom))
@@
     (effects (font (size 1 1)) (justify left bottom))
   )
+  (label "USB_VBUS2" (at 58.42 99.695 0)
+    (effects (font (size 1.27 1.27)) (justify left bottom))
+  )
   (label "SPI1_SCK" (at 137.16 172.085 180)

Commit message: Few changes
Connections:
- net B_m: now reaches BZ1.2 (+), Q1.3 (D), R6.1
- net ON_LED: now reaches D1.1 (K), R2.1
- net VDDA: now reaches C31.2, FB2.2, U4.8 (VDDA/VREF+)
- net BOOT0: now reaches JP1.1 (A), R3.1, U4.4 (PH3_BOOT0)
- net VFB: now reaches C30.2, JP2.2 (B), L3.1, U4.31 (VFBSMPS)
- net VLX: now reaches L3.2, U4.33 (VLXSMPS)
Other:
- moved on the sheet: BZ1, C30, D2, J10, J8, J9, JP1, R11, R3, R4
